File: Joystick.sch (KiCad schematic (older format))
At the start: 2 parts, among them J1 Conn_02x08_Counter_Clockwise, J2 DE9_Male_MountingHoles

Commit message: Associate footprints.
Parts:
- J1: footprint (none) -> Housings_DIP:DIP-16_W7.62mm_Socket; Description (none) -> CONN IC DIP SOCKET 16POS TIN; Digi-Key_PN (none) -> AE9992-ND; MPN (none) -> A 16-LC-TT
- J2: footprint (none) -> footprints:DSUB-9_Male_Horizontal_P2.77x2.84mm_EdgePinOffset7.70mm_Housed_MountingHolesOffset9.12mm; Description (none) -> CONN D-SUB PLUG 9POS R/A SOLDER; Digi-Key_PN (none) -> AE10968-ND; MPN (none) -> A-DS 09 A/KG-T2S
Changed lines of the file:
@@
 F 0 "J2" H 6200 4550 50  0000 C CNN
 F 1 "DE9_Male_MountingHoles" H 6200 4475 50  0000 C CNN
-F 2 "" H 6200 3900 50  0001 C CNN
+F 2 "footprints:DSUB-9_Male_Horizontal_P2.77x2.84mm_EdgePinOffset7.70mm_Housed_MountingHolesOffset9.12mm" H 6200 3900 50  0001 C CNN
 F 3 "" H 6200 3900 50  0001 C CNN
+F 4 "A-DS 09 A/KG-T2S" H 6200 3900 60  0001 C CNN "MPN"
+F 5 "CONN D-SUB PLUG 9POS R/A SOLDER" H 6200 3900 60  0001 C CNN "Description"
+F 6 "AE10968-ND" H 6200 3900 60  0001 C CNN "Digi-Key_PN"
 	1    6200 3900
 	1    0    0    -1
@@
 F 0 "J1" H 4150 4200 50  0000 C CNN
 F 1 "Conn_02x08_Counter_Clockwise" H 4150 3300 50  0000 C CNN
-F 2 "" H 4100 3800 50  0001 C CNN
+F 2 "Housings_DIP:DIP-16_W7.62mm_Socket" H 4100 3800 50  0001 C CNN
 F 3 "" H 4100 3800 50  0001 C CNN
+F 4 "A 16-LC-TT" H 4100 3800 60  0001 C CNN "MPN"
+F 5 "CONN IC DIP SOCKET 16POS TIN" H 4100 3800 60  0001 C CNN "Description"
+F 6 "AE9992-ND" H 4100 3800 60  0001 C CNN "Digi-Key_PN"
 	1    4100 3800
 	1    0    0    -1
